Commit message: Service Robot Project Files

File: my_robot/urdf/new_robot.xacro (robot description, xacro)
@@ -68,5 +68,5 @@
 		  	<origin xyz="0 0 0" rpy=" 0 0 -1.5707"/>
 		  	<geometry>
-		    	<box size="0.6 0.6 .1"/>
+		    	<box size="0.5 0.5 .1"/>
 		  	</geometry>
 		</collision>
@@ -74,5 +74,5 @@
 		  	<origin xyz="0 0 0" rpy=" 0 0 -1.5707"/>
 		  	<geometry>
-		    	<box size="0.5 0.5 .1"/>
+		    	<box size="0.4 0.4 .1"/>
 			</geometry>
 		</visual>
@@ -90,11 +90,11 @@
 			<origin xyz="0 0 0" rpy="1.5707 0 0"/>
 			<geometry>
-				<cylinder radius="0.1" length="0.05"/>
-			</geometry>
-		</visual>
-		<collision>
-			<origin xyz="0 0 0" rpy="1.5707 0 0"/>
-			<geometry>
-				<cylinder radius="0.1" length="0.05"/>
+				<cylinder radius="0.1" length="0.025"/>
+			</geometry>
+		</visual>
+		<collision>
+			<origin xyz="0 0 0" rpy="1.5707 0 0"/>
+			<geometry>
+				<cylinder radius="0.1" length="0.025"/>
 			</geometry>
 		</collision>
@@ -112,11 +112,11 @@
 			<origin xyz="0 0 0" rpy="1.5707 0 0"/>
 			<geometry>
-				<cylinder radius="0.1" length="0.05"/>
-			</geometry>
-		</visual>
-		<collision>
-			<origin xyz="0 0 0" rpy="1.5707 0 0"/>
-			<geometry>
-				<cylinder radius="0.1" length="0.05"/>
+				<cylinder radius="0.1" length="0.025"/>
+			</geometry>
+		</visual>
+		<collision>
+			<origin xyz="0 0 0" rpy="1.5707 0 0"/>
+			<geometry>
+				<cylinder radius="0.1" length="0.025"/>
 			</geometry>
 		</collision>
@@ -134,11 +134,11 @@
 			<origin xyz="0 0 0" rpy="1.5707 0 0"/>
 			<geometry>
-				<cylinder radius="0.1" length="0.05"/>
-			</geometry>
-		</visual>
-		<collision>
-			<origin xyz="0 0 0" rpy="1.5707 0 0"/>
-			<geometry>
-				<cylinder radius="0.1" length="0.05"/>
+				<cylinder radius="0.1" length="0.025"/>
+			</geometry>
+		</visual>
+		<collision>
+			<origin xyz="0 0 0" rpy="1.5707 0 0"/>
+			<geometry>
+				<cylinder radius="0.1" length="0.025"/>
 			</geometry>
 		</collision>
@@ -156,11 +156,11 @@
 			<origin xyz="0 0 0" rpy="1.5707 0 0"/>
 			<geometry>
-				<cylinder radius="0.1" length="0.05"/>
-			</geometry>
-		</visual>
-		<collision>
-			<origin xyz="0 0 0" rpy="1.5707 0 0"/>
-			<geometry>
-				<cylinder radius="0.1" length="0.05"/>
+				<cylinder radius="0.1" length="0.025"/>
+			</geometry>
+		</visual>
+		<collision>
+			<origin xyz="0 0 0" rpy="1.5707 0 0"/>
+			<geometry>
+				<cylinder radius="0.1" length="0.025"/>
 			</geometry>
 		</collision>
@@ -178,5 +178,5 @@
 			<origin xyz="0 0 0" rpy="0 0 0"/>
 			<geometry>
-				<cylinder radius="0.22" length="0.12"/>
+				<cylinder radius="0.15" length="0.12"/>
 			</geometry>
 		</visual>
@@ -184,5 +184,5 @@
 			<origin xyz="0 0 0" rpy="0 0 0"/>
 			<geometry>
-				<cylinder radius="0.22" length="0.12"/>
+				<cylinder radius="0.15" length="0.12"/>
 			</geometry>
 		</collision>
@@ -194,5 +194,5 @@
 	</joint>
 	<joint name="left_front_axis" type="continuous">
-		<origin xyz="0.2 0.278 0.02" rpy="0 0 0"/>
+		<origin xyz="0.14 0.218 0.02" rpy="0 0 0"/>
 		<child link="wheel_left_front"/>
 		<parent link="chassis"/>
@@ -202,5 +202,5 @@
 	</joint>
 	<joint name="left_back_axis" type="continuous">
-		<origin xyz="-0.2 0.278 0.02" rpy="0 0 0"/>
+		<origin xyz="-0.14 0.218 0.02" rpy="0 0 0"/>
 		<child link="wheel_left_back"/>
 		<parent link="chassis"/>
@@ -210,5 +210,5 @@
 	</joint>
 	<joint name="right_back_axis" type="continuous">
-		<origin xyz="-0.2 -0.278 0.02" rpy="0 0 0"/>
+		<origin xyz="-0.14 -0.218 0.02" rpy="0 0 0"/>
 		<child link="wheel_right_back"/>
 		<parent link="chassis"/>
@@ -218,5 +218,5 @@
 	</joint>
 	<joint name="right_front_axis" type="continuous">
-		<origin xyz="0.2 -0.278 0.02" rpy="0 0 0"/>
+		<origin xyz="0.14 -0.218 0.02" rpy="0 0 0"/>
 		<child link="wheel_right_front"/>
 		<parent link="chassis"/>
@@ -276,8 +276,15 @@
 	</link>
   <joint type="fixed" name="camera_joint">
-    <origin xyz="0.265 0 -0.03" rpy="0 0 0"/>
+    <origin xyz="0.215 0 -0.03" rpy="0 0 0"/>
     <child link="camera"/>
     <parent link="chassis"/>
     <axis xyz="0 1 0" rpy="0 0 0"/>
   </joint>
+  <joint name="camera_optical_joint" type="fixed">
+    <origin xyz="0 0 0" rpy="-1.5707 0 -1.5707"/>
+    <parent link="camera"/>
+    <child link="camera_link_optical"/>
+  </joint>
+  <link name="camera_link_optical">
+  </link>
 </robot>
